File: kicad/project/switching_board/switching_board.sch (KiCad schematic (older format))
At the start: 1 part

Commit message: FET
Parts:
- added F? (x4): Fuse, symbol Device:Fuse
- added J1, J? (x3): Output_conn, symbol Connector:Conn_01x02_Male
- added Q1, Q? (x3): n-mosfet, symbol Device:Q_NMOS_GDSD
- added R1, R? (x3): R(1) : 20 (V) / i = 1k, symbol Device:R
- added R2: R(3) : 4/(i * FET_num), symbol Device:R
- added R3, R? (x3): R(2) : R(1) * 10, symbol Device:R
- added SW1: emergency_switch, symbol Switch:SW_Push
- BT1: renamed from BT?; value Battery -> Battery(24v)
Connections:
- net VDD: now reaches BT1.1 (+)
- net VDD: now also F?.1, F?.1, F?.1, F?.1, SW1.1
- net GND: now reaches BT1.2 (-)
- net GND: now also Q1.3 (S), Q?.3 (S), Q?.3 (S), Q?.3 (S), R3.2, R?.2, R?.2, R?.2
- new net: Q1.1 (G), R1.1, R3.1
- new net: J1.1 (Pin_1), Q1.2 (D), Q1.4 (D)
- new net: R2.2, SW1.2
- new net: F?.2, J1.2 (Pin_2)
- new net: J?.1 (Pin_1), Q?.2 (D), Q?.4 (D) (x3)
- new net: F?.2, J?.2 (Pin_2) (x3)
- new net: Q?.1 (G), R?.1, R?.1 (x3)
- new net switch_signal: R1.2, R2.1, R?.2, R?.2, R?.2
Other:
- note added: "Carrent param \nVgs : 20 (V)\n"
- note added: "R(1) param\nQt : 50 (nC)\nt : 2500 (nsec)\ni = Qt/t = 0.02 (A)\n"
- note added: "absolute maximum ratings\nVds : 30 (V)\nVgs : 20 (V)\nId : 74 (A)\n"
- note added: "n-mosfet (name : IRL8113)\n1-gate\n2-drain\n3-source\n4-drain(backplate)"
- note added: "voltage step-down register\n from 24 (V) to 20 (V)\n"
