File: kicad/project/switching_board/_autosave-switching_board.sch (KiCad schematic (older format))
At the start: 35 parts, among them J1 Output_conn, J2 voltage_Output_conn, J3 Output_conn, J4 Output_conn, Q1 n-mosfet, Q2 n-mosfet, Q3 n-mosfet, Q4 n-mosfet, SW1 emergency_switch, U1 regulator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

Commit message: switching-board-v1.1.0
Parts:
- R1: value R(1) : 12 (V) / i = 1.2k -> R(1) : 12 (V) / i = 1k
- R10, R12, R7: value R(1) : 1.2k -> R(1) : 1k
- R11, R13, R8: value R(2) : 12k -> R(2) : 10k
- R3: value R(2) : R(1) * 10 = 12k -> R(2) : R(1) * 10 = 10k
Other:
- note added: "R(1) param\nQt : 58 (nC)\nt : 5000 (nsec)\ni = Qt/t = 0.0116 (A)\nR = V / i = 12 / 0.0116 = 1 (kOhm)\n"
- note removed: "R(1) param\nQt : 50 (nC)\nt : 5000 (nsec)\ni = Qt/t = 0.01 (A)\nR = V / i = 12 / 0.01 = 1.2 (kOhm)\n"
Changed lines of the file:
@@
 absolute maximum ratings\nVds : 30 (V)\nVgs : 20 (V)\nId : 74 (A)\n
 Text Notes 7050 1000 0    50   ~ 0
-R(1) param\nQt : 50 (nC)\nt : 5000 (nsec)\ni = Qt/t = 0.01 (A)\nR = V / i = 12 / 0.01 = 1.2 (kOhm)\n
+R(1) param\nQt : 58 (nC)\nt : 5000 (nsec)\ni = Qt/t = 0.0116 (A)\nR = V / i = 12 / 0.0116 = 1 (kOhm)\n
 $Comp
 L power:GND #PWR0101
@@
 P 1550 5700
 F 0 "R3" H 1400 5750 50  0001 L CNN
-F 1 "R(2) : R(1) * 10 = 12k" H 550 5650 50  0000 L CNN
+F 1 "R(2) : R(1) * 10 = 10k" H 550 5650 50  0000 L CNN
 F 2 "" V 1480 5700 50  0001 C CNN
 F 3 "~" H 1550 5700 50  0001 C CNN
@@
 P 1300 5450
 F 0 "R1" V 1093 5450 50  0001 C CNN
-F 1 "R(1) : 12 (V) / i = 1.2k" V 1200 5350 50  0000 C CNN
+F 1 "R(1) : 12 (V) / i = 1k" V 1200 5350 50  0000 C CNN
 F 2 "" V 1230 5450 50  0001 C CNN
 F 3 "~" H 1300 5450 50  0001 C CNN
@@
 P 3000 5700
 F 0 "R8" H 2850 5750 50  0001 L CNN
-F 1 "R(2) :  12k" H 2500 5700 50  0000 L CNN
+F 1 "R(2) :  10k" H 2500 5700 50  0000 L CNN
 F 2 "" V 2930 5700 50  0001 C CNN
 F 3 "~" H 3000 5700 50  0001 C CNN
@@
 P 2750 5450
 F 0 "R7" V 2543 5450 50  0001 C CNN
-F 1 "R(1) : 1.2k" V 2650 5400 50  0000 C CNN
+F 1 "R(1) : 1k" V 2650 5400 50  0000 C CNN
 F 2 "" V 2680 5450 50  0001 C CNN
 F 3 "~" H 2750 5450 50  0001 C CNN
@@
 P 6200 5700
 F 0 "R13" H 6050 5750 50  0001 L CNN
-F 1 "R(2) : 12k" H 5750 5700 50  0000 L CNN
+F 1 "R(2) : 10k" H 5750 5700 50  0000 L CNN
 F 2 "" V 6130 5700 50  0001 C CNN
 F 3 "~" H 6200 5700 50  0001 C CNN
@@
 P 5950 5450
 F 0 "R12" V 5743 5450 50  0001 C CNN
-F 1 "R(1) : 1.2k" V 5850 5450 50  0000 C CNN
+F 1 "R(1) : 1k" V 5850 5450 50  0000 C CNN
 F 2 "" V 5880 5450 50  0001 C CNN
 F 3 "~" H 5950 5450 50  0001 C CNN
@@
 P 4200 5450
 F 0 "R10" V 3993 5450 50  0001 C CNN
-F 1 "R(1) :  1.2k" V 4100 5400 50  0000 C CNN
+F 1 "R(1) :  1k" V 4100 5400 50  0000 C CNN
 F 2 "" V 4130 5450 50  0001 C CNN
 F 3 "~" H 4200 5450 50  0001 C CNN
@@
 P 4450 5700
 F 0 "R11" H 4300 5750 50  0001 L CNN
-F 1 "R(2) : 12k" H 4000 5700 50  0000 L CNN
+F 1 "R(2) : 10k" H 4000 5700 50  0000 L CNN
 F 2 "" V 4380 5700 50  0001 C CNN
 F 3 "~" H 4450 5700 50  0001 C CNN
